Commit message: Add optional mount joint to blackfly_s xacro macro
The macro defined the camera links but no joint attaching them to a host
robot, so it could only be used standalone (as in demo.urdf.xacro, where
${frame} is a root link). To weld the camera onto a vehicle URDF the
integrator previously had to add the mount joint by hand.

Add parent/mount_xyz/mount_rpy parameters. When parent is non-empty the macro
emits a fixed ${frame}_mount_joint from parent to ${frame}; when parent is
empty (the default) no joint is emitted and the standalone behaviour is
unchanged. Verified: demo.urdf.xacro still expands with ${frame} as root, and
supplying a parent produces a single well-formed mount joint.

Also correct two typos in the lens link that made its <inertial> block a
no-op: the element was misspelled <intertial> and used <mass values=...>
instead of <mass value=...>.

File: flir_camera_description/urdf/flir_blackfly_s.urdf.xacro (robot description, xacro)
@@ -5,9 +5,24 @@
         lens_{r, h, mass} are physical properties of the camera lens
         hfov, fps, width, height, format, near, and far are simulation
+        parent/mount_xyz/mount_rpy attach the camera to a host robot. Leave
+        parent empty (the default) to instantiate the camera standalone, in
+        which case ${frame} becomes a root link (see demo.urdf.xacro). Pass a
+        parent link name plus mount_xyz/mount_rpy to weld ${frame} onto a car
+        URDF (see docs/UQR_INTEGRATION.md).
     -->
     <xacro:macro name="flir_blackfly_s"
-        params="frame:=camera name:=camera camera_x:=0.047758 camera_y:=0.029 camera_z:=0.029 camera_mass:=0.03
-                lens_r:=0.016 lens_h:=0.04 lens_mass:= 0.05
+        params="frame:=camera name:=camera parent:='' mount_xyz:='0 0 0' mount_rpy:='0 0 0'
+                camera_x:=0.047758 camera_y:=0.029 camera_z:=0.029 camera_mass:=0.03
+                lens_r:=0.016 lens_h:=0.04 lens_mass:=0.05
                 hfov:=1.0471975512 fps:=30 width:=720 height:=540 format:=R8G8B8 near:=0.5 far:=300">
+        <!-- Optional mount joint welding the camera onto a host link. Only
+             created when a non-empty parent link is supplied. -->
+        <xacro:unless value="${parent == ''}">
+            <joint name="${frame}_mount_joint" type="fixed">
+                <origin xyz="${mount_xyz}" rpy="${mount_rpy}" />
+                <parent link="${parent}" />
+                <child link="${frame}" />
+            </joint>
+        </xacro:unless>
         <link name="${frame}">
         <inertial>
@@ -30,8 +45,8 @@
         </link>
         <link name="${frame}_lens">
-        <intertial>
-            <mass values="${lens_mass}" />
+        <inertial>
+            <mass value="${lens_mass}" />
             <inertia ixx="1e-6" ixy="0" ixz="0" iyy="1e-6" iyz="0" izz="1e-6" />
-        </intertial>
+        </inertial>
         <visual>
             <origin xyz="${lens_h/2} 0 0" rpy="0 1.5707 0" />
